File: RaspiCar_PCB2/RaspiCar_PCB1.kicad_pcb (KiCad board)
At the start: 2 copper layers, 63.5 x 54.5 mm, 14 parts

Commit message: RaspiCar_0.2
Added second PCB revision and full controller code
Parts:
- removed the PWR_GND at (175.8, 78.2)
- added C1: 1uF, Capacitor_SMD:C_Elec_5x5.4, F.Cu at (185.4, 88.9)
- added C2: 1uF, Capacitor_SMD:C_Elec_5x5.4, F.Cu at (190.5, 109.2)
- added PWR_GND: PWR_GND, Connector_PinHeader_2.54mm:PinHeader_1x02_P2.54mm_Vertical, F.Cu at (175.3, 78.7)
- added ServoPWR: ServoPWR/GND, Connector_PinHeader_2.54mm:PinHeader_1x02_P2.54mm_Vertical, F.Cu at (165.1, 78.7)
- renumbered L293D to L293D1, Raspi_Logic to Raspi_Logic1, Raspi_PWR to Raspi_PWR1
Routing:
- net GND: track 23.5 -> 50.8 mm, vias 8 -> 7
- net +7.5V: track 19.3 -> 40.8 mm
- net +5V: track 50.7 -> 62.7 mm
- net Net-(L293D1-Pad14): track 13.4 -> 17.8 mm
- net Net-(L293D1-Pad11): track 23.1 -> 26.4 mm
- net Net-(L293D1-Pad6): track 27.2 -> 29.8 mm
Other:
- board text added: "PWR-GND"
- board text added: "Raspberry Pi RC Car - PCB_2 Benjamin Bega - 2022"
- board text removed: "Raspberry Pi RC Car - PCB_1 Benjamin Bega -2022"
