File: RaspiCar_PCB2/RaspiCar_PCB1.kicad_sch (KiCad schematic)
At the start: 14 parts

Commit message: RaspiCar_0.2
Added second PCB revision and full controller code
Parts:
- added C1, C2: 1uF, Capacitor_SMD:C_Elec_5x5.4, symbol Device:C
- added ServoPWR1: ServoPWR/GND, Connector_PinHeader_2.54mm:PinHeader_1x02_P2.54mm_Vertical, symbol Connector:Conn_01x02_Male
- PWR_GND1: value PWR_GND -> (none); footprint Connector_AMASS:AMASS_XT60-F_1x02_P7.20mm_Vertical -> Connector_PinHeader_2.54mm:PinHeader_1x02_P2.54mm_Vertical
Connections:
- net +5V: now also C2.1
- net +7.5V: now also C1.1, ServoPWR1.2 (Pin_2)
- net GND: now also C1.2, C2.2, ServoPWR1.1 (Pin_1)
Other:
- moved on the sheet: H1, H2, H3, H4
